File: Penny_triple/Penny_triple.kicad_sch (KiCad schematic)
At the start: 3 parts, among them J1 USB3_A, J2 USB_C_Receptacle, J3 USB3_A

Commit message: v0.2 circuit was created
Parts:
- removed J2: USB_C_Receptacle, symbol Connector:USB_C_Receptacle
- added C? (x2): 120 uF, Capacitor_THT:CP_Radial_D6.3mm_P2.50mm, symbol Device:C_Polarized
- added C? (x2): 2.2, Capacitor_SMD:C_0603_1608Metric_Pad1.08x0.95mm_HandSolder, symbol Device:C
- added C? (x2): 0.1, Capacitor_SMD:C_0603_1608Metric_Pad1.08x0.95mm_HandSolder, symbol Device:C
- added J?: Conn_01x06_Female, Connector_PinSocket_2.54mm:PinSocket_1x06_P2.54mm_Vertical, symbol Connector:Conn_01x06_Female
- added J? (x2): Conn_01x02_Female, Connector_PinSocket_2.54mm:PinSocket_1x02_P2.54mm_Vertical, symbol Connector:Conn_01x02_Female
- added R? (x4): 10k, Resistor_SMD:R_0603_1608Metric_Pad0.98x0.95mm_HandSolder, symbol Device:R
- added R? (x2): R, Resistor_SMD:R_0603_1608Metric_Pad0.98x0.95mm_HandSolder, symbol Device:R
- added U? (x2): TPS2553, Package_TO_SOT_SMD:SOT-23-6_Handsoldering, symbol Shield_Emergent:TPS2553
- added X?: USB_C_24pins, Shield1:FPC_12, symbol Shield1:USB_C_24pins
Connections:
- net VBUS1: now reaches J1.1 (VBUS)
- net VBUS1: now also C?.1, U?.1 (In)
- net Earth: now reaches J1.10 (SHIELD)
- net Earth: now also J3.10 (SHIELD), X?.S1 (SHIELD), X?.S2 (SHIELD), X?.S3 (SHIELD), X?.S4 (SHIELD)
- net GND1: now reaches J1.4 (GND)
- net GND1: now also J1.7 (DRAIN), J3.4 (GND), J3.7 (DRAIN), C?.2, C?.2, C?.2, C?.2, C?.2, C?.2, J?.2 (Pin_2), J?.2 (Pin_2), J?.4 (Pin_4), R?.2, R?.2, U?.2 (GND), U?.2 (GND), X?.A1 (GND), X?.A12 (GND), X?.B1 (GND), X?.B12 (GND)
- net RX1-: now reaches J1.5 (SSRX-)
- net RX1-: now also X?.B10 (RX1-)
- net RX1+: now reaches J1.6 (SSRX+)
- net RX1+: now also X?.B11 (RX1+)
- net TX1-: now reaches J1.8 (SSTX-)
- net TX1-: now also X?.A3 (TX1-)
- net TX1+: now reaches J1.9 (SSTX+)
- net TX1+: now also X?.A2 (TX1+)
- net VBUS2: now reaches J3.1 (VBUS)
- net VBUS2: now also C?.1, U?.1 (In)
- net RX2-: now reaches J3.5 (SSRX-)
- net RX2-: now also X?.A10 (RX2-)
- net RX2+: now reaches J3.6 (SSRX+)
- net RX2+: now also X?.A11 (RX2+)
- net TX2-: now reaches J3.8 (SSTX-)
- net TX2-: now also X?.B3 (TX2-)
- net TX2+: now reaches J3.9 (SSTX+)
- net TX2+: now also X?.B2 (TX2+)
- new net: R?.1, U?.5 (ILIM) (x2)
- new net +3V3: J?.3 (Pin_3), R?.1, R?.1, R?.2, R?.2
- new net EN1: J?.1 (Pin_1), R?.2, U?.3 (En)
- new net EN2: J?.5 (Pin_5), R?.2, U?.3 (En)
- new net FLT1: J?.2 (Pin_2), R?.1, U?.4 (FLT)
- new net FLT2: J?.6 (Pin_6), R?.1, U?.4 (FLT)
- new net Vout1: C?.1, C?.1, J?.1 (Pin_1), U?.6 (OUT), X?.A4 (VBUS), X?.B9 (VBUS)
- new net Vout2: C?.1, C?.1, J?.1 (Pin_1), U?.6 (OUT), X?.A9 (VBUS), X?.B4 (VBUS)
Other:
- moved on the sheet: J3

Commit message: v0.3 The circuit was complected
Parts:
- removed J?: Conn_01x06_Female, Connector_PinSocket_2.54mm:PinSocket_1x06_P2.54mm_Vertical, symbol Connector:Conn_01x06_Female
- added J?: Conn_02x06_Odd_Even, Connector_PinHeader_2.54mm:PinHeader_2x06_P2.54mm_Vertical, symbol Connector_Generic:Conn_02x06_Odd_Even
Connections:
- net +3V3: now also J?.1 (Pin_1), J?.2 (Pin_2)
- net EN1: now also J?.3 (Pin_3)
- net EN2: now also J?.4 (Pin_4)
- net FLT1: now also J?.7 (Pin_7)
- net FLT2: now also J?.8 (Pin_8)
- net GND1: now also J?.5 (Pin_5), J?.6 (Pin_6)
- net B3: now reaches X?.A5 (CC1)
- net B3: now also J?.10 (Pin_10)
- net B1: now reaches X?.A8 (SBU1)
- net B1: now also J?.12 (Pin_12)
- net B4: now reaches X?.B5 (CC2)
- net B4: now also J?.9 (Pin_9)
- net B2: now reaches X?.B8 (SBU2)
- net B2: now also J?.11 (Pin_11)
Other:
- moved on the sheet: J?, X?

Commit message: v0.4 circuit was completed
Parts:
- removed J3: USB3_A, symbol Connector:USB3_A
- added C? (x4): 2.2, Capacitor_SMD:C_0603_1608Metric_Pad1.08x0.95mm_HandSolder, symbol Device:C
- added D?: PMEG2020EH, Diode_SMD:D_SOD-123F, symbol Diode:PMEG2020EH
- added J? (x3): Conn_01x02_Female, Connector_PinSocket_2.54mm:PinSocket_1x02_P2.54mm_Vertical, symbol Connector:Conn_01x02_Female
- added J?: USB3_A, symbol Connector:USB3_A
- added R? (x5): 0, Resistor_SMD:R_0201_0603Metric_Pad0.64x0.40mm_HandSolder, symbol Device:R
- added U? (x2): LM7805_TO220, Package_TO_SOT_THT:TO-220-3_Vertical, symbol Regulator_Linear:LM7805_TO220
Connections:
- net VBUS2 is gone; now on net +5V: C?.1, U?.1 (In)
- net +3V3: now also C?.1, U?.3 (VO)
- net Earth: now also J1.11 (SHIELD), J?.10 (SHIELD), J?.11 (SHIELD), R?.1, R?.1, R?.1
- net GND1: now also C?.2, C?.2, C?.2, C?.2, J?.2 (Pin_2), J?.2 (Pin_2), J?.4 (GND), J?.7 (DRAIN), R?.2, R?.2, U?.2 (GND), U?.2 (GND); no longer X?.A1 (GND), X?.A12 (GND), X?.B1 (GND), X?.B12 (GND)
- net RX2+: now also J?.6 (SSRX+)
- net RX2-: now also J?.5 (SSRX-)
- net TX2+: now also J?.9 (SSTX+)
- net TX2-: now also J?.8 (SSTX-)
- net at X?.A6 (D+): now also X?.B6 (D+), J?.2 (Pin_2)
- net at X?.A7 (D-): now also X?.B7 (D-), J?.1 (Pin_1)
- net VBUS1 renamed +5V
- net +5V: now also C?.1, D?.1 (K), J?.1 (Pin_1), R?.2, R?.2, U?.1 (VI); no longer J1.1 (VBUS)
- new net: J?.1 (VBUS), R?.1
- new net: J1.1 (VBUS), R?.1
- new net: R?.2, X?.A1 (GND), X?.A12 (GND), X?.B1 (GND), X?.B12 (GND)
- new net: C?.1, D?.2 (A), U?.3 (VO)
- new net +12V: C?.1, J?.1 (Pin_1), U?.1 (VI)
Other:
- moved on the sheet: J?, R?, X?
